File: schematic/PowerBoard.kicad_pcb (KiCad board)
At the start: 2 copper layers, 20 parts, among them J1 ToResistor, Q1 IRLB8721PBF, U1 PAM2423A

Commit message: Completed pcb design
Parts:
- added REF**: MountingHole_3.2mm_M3, Mounting_Holes:MountingHole_3.2mm_M3, F.Cu at (113.0, 53.3)
- added REF**: MountingHole_3.2mm_M3, Mounting_Holes:MountingHole_3.2mm_M3, F.Cu at (186.7, 53.3)
- added REF**: MountingHole_3.2mm_M3, Mounting_Holes:MountingHole_3.2mm_M3, F.Cu at (109.2, 139.1)
- added REF**: MountingHole_3.2mm_M3, Mounting_Holes:MountingHole_3.2mm_M3, F.Cu at (189.2, 139.1)
- moved J1 88.0 mm to (112.3, 113.3), turned to 180 degrees
- moved Q1 54.5 mm to (124.0, 115.8), turned to 270 degrees
- moved D2 49.8 mm to (123.4, 106.7), turned to 180 degrees
- moved R4 46.6 mm to (122.9, 109.7), turned to 180 degrees
- moved C1 35.3 mm to (156.0, 70.1)
- moved R1 29.3 mm to (133.1, 94.0)
- moved R2 28.9 mm to (133.1, 97.5), turned to 180 degrees
- moved U1 27.4 mm to (146.3, 87.9), turned to 180 degrees
- moved C6 16.5 mm to (133.1, 90.4)
- moved D1 16.0 mm to (133.1, 82.3), turned to 270 degrees
- moved C5 14.5 mm to (158.0, 85.9)
- moved C8 12.9 mm to (139.2, 70.1), turned to 180 degrees
- moved C2 12.8 mm to (152.9, 78.2)
- moved C3 12.0 mm to (164.1, 88.9)
- moved C7 9.88 mm to (141.2, 78.2), turned to 180 degrees
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Connections:
- Q1 pad 1: Pri_Deploy -> LineDeploymentDevice
- Q1 pad 3: GND -> Pri_Deploy
- Q1 pad 4: (no net) -> GND
- Q1 pad 5: (no net) -> LineDeploymentDevice
- Q1 pad 6: (no net) -> LineDeploymentDevice
- R4 pad 1: Net-(R4-Pad1) -> Pri_Deploy
Routing:
- net Pri_Deploy: track 0.00 -> 71.8 mm
- net +5V: track 0.00 -> 48.1 mm, vias 0 -> 2
- net +8V: track 0.00 -> 41.6 mm
- net GND: track 0.00 -> 21.2 mm, vias 0 -> 4
- net Net-(D1-Pad2): track 0.00 -> 16.1 mm
- net LineDeploymentDevice: track 0.00 -> 15.7 mm
- net Net-(R1-Pad2): track 0.00 -> 15.4 mm
- net Net-(C5-Pad1): track 0.00 -> 11.5 mm, vias 0 -> 2
- net Net-(C6-Pad2): track 0.00 -> 10.8 mm
- net Net-(C3-Pad1): track 0.00 -> 4.15 mm
- net Net-(D2-Pad2): track 0.00 -> 3.20 mm
- added copper zone on B.Cu, net +5V
- added copper zone on F.Cu, net GND
Other:
- board outline added: 90.2 x 95.9 mm
- board text added: "CySat 1 - Power Board v1"

Commit message: Playing with via values to get advanced circuits to take it
Connections:
- H2 pad 19: Net-(H2-Pad19) -> +8V
- H2 pad 20: Net-(H2-Pad20) -> +8V
Routing:
- net +8V: track 41.6 -> 58.9 mm
- net GND: track 21.2 -> 37.6 mm, vias 4 -> 1
Other:
- net class Default: clearance 0.2 -> 0.2032; via_dia 0.6 -> 0.508; via_drill 0.4 -> 0.4318
- rule trace_clearance: 0.2 -> 0.2032
- board text added: "+"

Commit message: Update check
Parts:
- added D3: LED, LEDs:LED_0805, F.Cu at (123.8, 122.2)
- added J2: ToResistor, Pin_Headers:Pin_Header_Straight_1x02_Pitch2.54mm, F.Cu at (112.3, 126.0)
- added LOGO: , motherboard:LOGO, F.Cu at (145.7, 111.8)
- added Q2: IRLB8721PBF, TO_SOT_Packages_SMD:SOT-666, F.Cu at (122.5, 130.2)
- added R5: 51, Resistors_SMD:R_0805, F.Cu at (123.4, 125.2)
Connections:
- J1 pad 1: LineDeploymentDevice -> SecondaryLineDeploymentDevice
- Q1 pad 1: LineDeploymentDevice -> (no net)
- Q1 pad 2: LineDeploymentDevice -> SecondaryLineDeploymentDevice
- Q1 pad 5: LineDeploymentDevice -> (no net)
- Q1 pad 6: LineDeploymentDevice -> (no net)
Routing:
- net Pri_Deploy: track 72.1 -> 116.9 mm
- net SecondaryLineDeploymentDevice: track 0.00 -> 15.7 mm
- net Net-(D3-Pad2): track 0.00 -> 2.99 mm
- net GND: track 37.6 -> 40.1 mm
