File: schematic/PowerBoard.sch (KiCad schematic (older format))
At the start: 14 parts, among them U1 PAM2423A

Commit message: Added mosfet
Parts:
- added H? (x2): CONN_02X26, motherboard:CSK_Header, symbol CONN_02X26
- added J1: ToResistor, symbol Conn_01x02
- added Q1: IRLB8721PBF, TO_SOT_Packages_THT:TO-220_Vertical, symbol IRLB8721PBF
- C1: footprint (none) -> Capacitors_SMD:CP_Elec_8x10.5
- C2, C3, C4, C5, C6, C7: footprint (none) -> Capacitors_SMD:C_0805
- C8: footprint (none) -> Capacitors_SMD:CP_Elec_8x10
- D1: footprint (none) -> Diodes_SMD:D_SMC
- L1: footprint (none) -> Inductors_SMD:L_0805
- R1, R2, R3: footprint (none) -> Resistors_SMD:R_0805
- U1: footprint (none) -> Housings_SOIC:HTSOP-8-1EP_3.9x4.9mm_Pitch1.27mm
Connections:
- net labels added: +5V, LineDeploymentDevice, RADIO_RR_P, Switch
- wire segments 19 -> 43
- no-connect marks 0 -> 90
Other:
- note added: "H1"
- note added: "H2"
- moved on the sheet: C1, C2, C3, C4, C5, C6, C7, C8, D1, L1, R1, R2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

Commit message: Started Schematic
Parts:
- added D2: LED, LEDs:LED_0805, symbol LED
- added R4: 51, Resistors_SMD:R_0805, symbol R
- J1: footprint (none) -> Pin_Headers:Pin_Header_Straight_1x02_Pitch2.54mm
- gave numbers to parts that had none: 2
Connections:
- net labels added: Pri_Deploy, Sec_Deploy
- net labels removed: Switch
- wire segments 43 -> 46
- no-connect marks 90 -> 88
Other:
- moved on the sheet: Q1
Changed lines of the file:
@@
 $EndDescr
 $Comp
-L +8V #PWR17
+L +8V #PWR01
 U 1 1 5B2D431C
 P 9400 2600
-F 0 "#PWR17" H 9400 2450 50  0001 C CNN
+F 0 "#PWR01" H 9400 2450 50  0001 C CNN
 F 1 "+8V" H 9400 2740 50  0000 C CNN
 F 2 "" H 9400 2600 50  0001 C CNN
@@
 	7150 2900 7150 2850
 $Comp
-L GND #PWR11
+L GND #PWR02
 U 1 1 5B2D4448
 P 7150 2850
-F 0 "#PWR11" H 7150 2600 50  0001 C CNN
+F 0 "#PWR02" H 7150 2600 50  0001 C CNN
 F 1 "GND" H 7150 2700 50  0000 C CNN
 F 2 "" H 7150 2850 50  0001 C CNN
@@
 $EndComp
 $Comp
-L GND #PWR10
+L GND #PWR03
 U 1 1 5B2D4507
 P 7000 3300
-F 0 "#PWR10" H 7000 3050 50  0001 C CNN
+F 0 "#PWR03" H 7000 3050 50  0001 C CNN
 F 1 "GND" H 7000 3150 50  0000 C CNN
 F 2 "" H 7000 3300 50  0001 C CNN
@@
 	7200 4200 6900 4200
 $Comp
-L GND #PWR9
+L GND #PWR04
 U 1 1 5B2D4619
 P 6900 4200
-F 0 "#PWR9" H 6900 3950 50  0001 C CNN
+F 0 "#PWR04" H 6900 3950 50  0001 C CNN
 F 1 "GND" H 6900 4050 50  0000 C CNN
 F 2 "" H 6900 4200 50  0001 C CNN
@@
 $EndComp
 $Comp
-L GND #PWR14
+L GND #PWR05
 U 1 1 5B2D473B
 P 8850 3450
-F 0 "#PWR14" H 8850 3200 50  0001 C CNN
+F 0 "#PWR05" H 8850 3200 50  0001 C CNN
 F 1 "GND" H 8850 3300 50  0000 C CNN
 F 2 "" H 8850 3450 50  0001 C CNN
@@
 Connection ~ 8850 3100
 $Comp
-L GND #PWR12
+L GND #PWR06
 U 1 1 5B2D4783
 P 8100 3200
-F 0 "#PWR12" H 8100 2950 50  0001 C CNN
+F 0 "#PWR06" H 8100 2950 50  0001 C CNN
 F 1 "GND" H 8100 3050 50  0000 C CNN
 F 2 "" H 8100 3200 50  0001 C CNN
@@
 $EndComp
 $Comp
-L GND #PWR8
+L GND #PWR07
 U 1 1 5B2D47DE
 P 6700 2900
-F 0 "#PWR8" H 6700 2650 50  0001 C CNN
+F 0 "#PWR07" H 6700 2650 50  0001 C CNN
 F 1 "GND" H 6700 2750 50  0000 C CNN
 F 2 "" H 6700 2900 50  0001 C CNN
@@
 $EndComp
 $Comp
-L GND #PWR7
+L GND #PWR08
 U 1 1 5B2D483D
 P 6400 2900
-F 0 "#PWR7" H 6400 2650 50  0001 C CNN
+F 0 "#PWR08" H 6400 2650 50  0001 C CNN
 F 1 "GND" H 6400 2750 50  0000 C CNN
 F 2 "" H 6400 2900 50  0001 C CNN
@@
 $EndComp
 $Comp
-L GND #PWR15
+L GND #PWR09
 U 1 1 5B2D48A2
 P 9050 2900
-F 0 "#PWR15" H 9050 2650 50  0001 C CNN
+F 0 "#PWR09" H 9050 2650 50  0001 C CNN
 F 1 "GND" H 9050 2750 50  0000 C CNN
 F 2 "" H 9050 2900 50  0001 C CNN
@@
 $EndComp
 $Comp
-L GND #PWR16
+L GND #PWR010
 U 1 1 5B2D4909
 P 9300 2900
-F 0 "#PWR16" H 9300 2650 50  0001 C CNN
+F 0 "#PWR010" H 9300 2650 50  0001 C CNN
 F 1 "GND" H 9300 2750 50  0000 C CNN
 F 2 "" H 9300 2900 50  0001 C CNN
@@
 $EndComp
 $Comp
-L GND #PWR13
+L GND #PWR011
 U 1 1 5B2D4939
 P 8450 3700
-F 0 "#PWR13" H 8450 3450 50  0001 C CNN
+F 0 "#PWR011" H 8450 3450 50  0001 C CNN
 F 1 "GND" H 8450 3550 50  0000 C CNN
 F 2 "" H 8450 3700 50  0001 C CNN
@@
 L IRLB8721PBF Q1
 U 1 1 5B33FF0C
-P 9050 5400
-F 0 "Q1" H 9300 5475 50  0000 L CNN
-F 1 "IRLB8721PBF" H 9300 5400 50  0000 L CNN
-F 2 "TO_SOT_Packages_THT:TO-220_Vertical" H 9300 5325 50  0001 L CIN
-F 3 "" H 9050 5400 50  0001 L CNN
-	1    9050 5400
-	1    0    0    -1
-$EndComp
-$Comp
-L GND #PWR5
+P 9050 5600
+F 0 "Q1" H 9300 5675 50  0000 L CNN
+F 1 "IRLB8721PBF" H 9300 5600 50  0000 L CNN
+F 2 "TO_SOT_Packages_THT:TO-220_Vertical" H 9300 5525 50  0001 L CIN
+F 3 "" H 9050 5600 50  0001 L CNN
+	1    9050 5600
+	1    0    0    -1
+$EndComp
+$Comp
+L GND #PWR012
 U 1 1 5B3400DC
-P 9150 5600
-F 0 "#PWR5" H 9150 5350 50  0001 C CNN
-F 1 "GND" H 9150 5450 50  0000 C CNN
-F 2 "" H 9150 5600 50  0001 C CNN
-F 3 "" H 9150 5600 50  0001 C CNN
-	1    9150 5600
-	1    0    0    -1
-$EndComp
-Wire Wire Line
-	9150 5200 9500 5200
+P 9150 5800
+F 0 "#PWR012" H 9150 5550 50  0001 C CNN
+F 1 "GND" H 9150 5650 50  0000 C CNN
+F 2 "" H 9150 5800 50  0001 C CNN
+F 3 "" H 9150 5800 50  0001 C CNN
+	1    9150 5800
+	1    0    0    -1
+$EndComp
+Wire Wire Line
+	9150 5400 9500 5400
 Text GLabel 9050 4850 2    60   Input ~ 0
 LineDeploymentDevice
 $Comp
-L +5V #PWR4
+L +5V #PWR013
 U 1 1 5B353A83
 P 9050 4750
-F 0 "#PWR4" H 9050 4600 50  0001 C CNN
+F 0 "#PWR013" H 9050 4600 50  0001 C CNN
 F 1 "+5V" H 9050 4890 50  0000 C CNN
 F 2 "" H 9050 4750 50  0001 C CNN
@@
 F 0 "J1" H 8850 4950 50  0000 C CNN
 F 1 "ToResistor" H 8850 4650 50  0000 C CNN
-F 2 "" H 8850 4850 50  0001 C CNN
+F 2 "Pin_Headers:Pin_Header_Straight_1x02_Pitch2.54mm" H 8850 4850 50  0001 C CNN
 F 3 "" H 8850 4850 50  0001 C CNN
 	1    8850 4850
@@
 H1
 $Comp
-L CONN_02X26 H?
+L CONN_02X26 H1
 U 1 1 5B3547F5
 P 9150 9600
-F 0 "H?" H 9150 10950 50  0000 C CNN
+F 0 "H1" H 9150 10950 50  0000 C CNN
 F 1 "CONN_02X26" V 9150 9600 50  0000 C CNN
 F 2 "motherboard:CSK_Header" H 9150 8900 50  0001 C CNN
@@
 H2
 $Comp
-L CONN_02X26 H?
+L CONN_02X26 H2
 U 1 1 5B3547F6
 P 10750 9600
-F 0 "H?" H 10750 10950 50  0000 C CNN
+F 0 "H2" H 10750 10950 50  0000 C CNN
 F 1 "CONN_02X26" V 10750 9600 50  0000 C CNN
 F 2 "motherboard:CSK_Header" H 10750 8900 50  0001 C CNN
@@
 Connection ~ 10450 8750
 $Comp
-L GND #PWR?
+L GND #PWR014
 U 1 1 5B354802
 P 10300 8800
-F 0 "#PWR?" H 10300 8550 50  0001 C CNN
+F 0 "#PWR014" H 10300 8550 50  0001 C CNN
 F 1 "GND" H 10300 8650 50  0000 C CNN
 F 2 "" H 10300 8800 60  0000 C CNN
@@
 	11000 8950 11200 8950
 $Comp
-L GND #PWR?
+L GND #PWR015
 U 1 1 5B354803
 P 11200 9000
-F 0 "#PWR?" H 11200 8750 50  0001 C CNN
+F 0 "#PWR015" H 11200 8750 50  0001 C CNN
 F 1 "GND" H 11200 8850 50  0000 C CNN
 F 2 "" H 11200 9000 60  0000 C CNN
@@
 NoConn ~ 11000 9450
 $Comp
-L +5V #PWR?
+L +5V #PWR016
 U 1 1 5B354804
 P 10300 9450
-F 0 "#PWR?" H 10300 9300 50  0001 C CNN
+F 0 "#PWR016" H 10300 9300 50  0001 C CNN
 F 1 "+5V" H 10300 9590 50  0000 C CNN
 F 2 "" H 10300 9450 60  0000 C CNN
@@
 $EndComp
 $Comp
-L +5V #PWR?
+L +5V #PWR017
 U 1 1 5B354805
 P 11200 9450
-F 0 "#PWR?" H 11200 9300 50  0001 C CNN
+F 0 "#PWR017" H 11200 9300 50  0001 C CNN
 F 1 "+5V" H 11200 9590 50  0000 C CNN
 F 2 "" H 11200 9450 60  0000 C CNN
@@
 	10300 9550 10500 9550
 $Comp
-L +3.3V #PWR?
+L +3.3V #PWR018
 U 1 1 5B354806
 P 10100 9600
-F 0 "#PWR?" H 10100 9450 50  0001 C CNN
+F 0 "#PWR018" H 10100 9450 50  0001 C CNN
 F 1 "+3.3V" H 10100 9740 50  0000 C CNN
 F 2 "" H 10100 9600 60  0000 C CNN
@@
 	10100 9650 10100 9600
 $Comp
-L +3.3V #PWR?
+L +3.3V #PWR019
 U 1 1 5B354807
 P 11400 9600
-F 0 "#PWR?" H 11400 9450 50  0001 C CNN
+F 0 "#PWR019" H 11400 9450 50  0001 C CNN
 F 1 "+3.3V" H 11400 9740 50  0000 C CNN
 F 2 "" H 11400 9600 60  0000 C CNN
@@
 NoConn ~ 9400 10750
 NoConn ~ 11000 8450
-Text GLabel 8850 5450 0    60   Input ~ 0
-Switch
-$Comp
-L PWR_FLAG #FLG1
+$Comp
+L PWR_FLAG #FLG020
 U 1 1 5B33FC3C
 P 850 7250
-F 0 "#FLG1" H 850 7325 50  0001 C CNN
+F 0 "#FLG020" H 850 7325 50  0001 C CNN
 F 1 "PWR_FLAG" H 850 7400 50  0000 C CNN
 F 2 "" H 850 7250 50  0001 C CNN
@@
 $EndComp
 $Comp
-L +5V #PWR1
+L +5V #PWR021
 U 1 1 5B33FC0C
 P 850 7250
-F 0 "#PWR1" H 850 7100 50  0001 C CNN
+F 0 "#PWR021" H 850 7100 50  0001 C CNN
 F 1 "+5V" H 850 7390 50  0000 C CNN
 F 2 "" H 850 7250 50  0001 C CNN
@@
 $EndComp
 $Comp
-L PWR_FLAG #FLG2
+L PWR_FLAG #FLG022
 U 1 1 5B2D6AAB
 P 1300 7250
-F 0 "#FLG2" H 1300 7325 50  0001 C CNN
+F 0 "#FLG022" H 1300 7325 50  0001 C CNN
 F 1 "PWR_FLAG" H 1300 7400 50  0000 C CNN
 F 2 "" H 1300 7250 50  0001 C CNN
@@
 $EndComp
 $Comp
-L +8V #PWR2
+L +8V #PWR023
 U 1 1 5B2D6A7B
 P 1300 7250
-F 0 "#PWR2" H 1300 7100 50  0001 C CNN
+F 0 "#PWR023" H 1300 7100 50  0001 C CNN
 F 1 "+8V" H 1300 7390 50  0000 C CNN
 F 2 "" H 1300 7250 50  0001 C CNN
@@
 $EndComp
 $Comp
-L PWR_FLAG #FLG3
+L PWR_FLAG #FLG024
 U 1 1 5B2D69BF
 P 1750 7250
-F 0 "#FLG3" H 1750 7325 50  0001 C CNN
+F 0 "#FLG024" H 1750 7325 50  0001 C CNN
 F 1 "PWR_FLAG" H 1750 7400 50  0000 C CNN
 F 2 "" H 1750 7250 50  0001 C CNN
@@
 $EndComp
 $Comp
-L +3.3V #PWR3
+L +3.3V #PWR025
 U 1 1 5B2D698F
 P 1750 7250
-F 0 "#PWR3" H 1750 7100 50  0001 C CNN
+F 0 "#PWR025" H 1750 7100 50  0001 C CNN
 F 1 "+3.3V" H 1750 7390 50  0000 C CNN
 F 2 "" H 1750 7250 50  0001 C CNN
@@
 	1    0    0    -1
 $EndComp
-Text GLabel 9500 5200 2    60   Input ~ 0
+Text GLabel 9500 5400 2    60   Input ~ 0
 LineDeploymentDevice
 $Comp
@@
 $EndComp
 $Comp
-L +5V #PWR?
+L +5V #PWR026
 U 1 1 5B35A9A0
 P 6200 2600
-F 0 "#PWR?" H 6200 2450 50  0001 C CNN
+F 0 "#PWR026" H 6200 2450 50  0001 C CNN
 F 1 "+5V" H 6200 2740 50  0000 C CNN
 F 2 "" H 6200 2600 50  0001 C CNN
@@
 NoConn ~ 11000 8550
 NoConn ~ 11000 8350
-NoConn ~ 10500 8350
 NoConn ~ 10500 8450
 NoConn ~ 10500 8550
@@
 NoConn ~ 8900 8550
 NoConn ~ 8900 8450
-NoConn ~ 8900 8350
 NoConn ~ 9400 8350
 NoConn ~ 9400 8450
@@
 NoConn ~ 9400 10650
 NoConn ~ 9400 9950
+Wire Wire Line
+	8900 5650 8900 5850
+Wire Wire Line
+	8900 5850 8800 5850
+$Comp
+L R R4
+U 1 1 5B36576A
+P 8650 5850
+F 0 "R4" V 8730 5850 50  0000 C CNN
+F 1 "51" V 8650 5850 50  0000 C CNN
+F 2 "Resistors_SMD:R_0805" V 8580 5850 50  0001 C CNN
+F 3 "" H 8650 5850 50  0001 C CNN
+	1    8650 5850
+	0    1    1    0
+$EndComp
+$Comp
+L LED D2
+U 1 1 5B3657B9
+P 8350 5850
+F 0 "D2" H 8350 5950 50  0000 C CNN
+F 1 "LED" H 8350 5750 50  0000 C CNN
+F 2 "LEDs:LED_0805" H 8350 5850 50  0001 C CNN
+F 3 "" H 8350 5850 50  0001 C CNN
+	1    8350 5850
+	1    0    0    -1
+$EndComp
+$Comp
+L GND #PWR027
+U 1 1 5B365800
+P 8200 5850
+F 0 "#PWR027" H 8200 5600 50  0001 C CNN
+F 1 "GND" H 8200 5700 50  0000 C CNN
+F 2 "" H 8200 5850 50  0001 C CNN
+F 3 "" H 8200 5850 50  0001 C CNN
+	1    8200 5850
+	0    1    1    0
+$EndComp
+Text GLabel 8900 8350 0    60   Input ~ 0
+Pri_Deploy
+Text GLabel 10500 8350 0    60   Input ~ 0
+Sec_Deploy
+Wire Wire Line
+	8450 5650 8850 5650
+Text GLabel 8450 5650 0    60   Input ~ 0
+Pri_Deploy
+Text GLabel 8600 5650 1    60   Input ~ 0
+Sec_Deploy
+Connection ~ 8900 5650
+Connection ~ 8800 5850
 $EndSCHEMATC

Commit message: Completed pcb design
Parts:
- J1: symbol Conn_01x02 -> CONN_01X02
Changed lines of the file:
@@
 EESchema Schematic File Version 2
+LIBS:PowerBoard-rescue
 LIBS:power
 LIBS:device
@@
 LIBS:contrib
 LIBS:valves
+LIBS:pam
 LIBS:PowerBoard-cache
-LIBS:motherboard-cache
 EELAYER 25 0
 EELAYER END
@@
 Wire Wire Line
 	9150 5400 9500 5400
-Text GLabel 9050 4850 2    60   Input ~ 0
+Text GLabel 9050 4900 2    60   Input ~ 0
 LineDeploymentDevice
 $Comp
 L +5V #PWR013
 U 1 1 5B353A83
-P 9050 4750
-F 0 "#PWR013" H 9050 4600 50  0001 C CNN
-F 1 "+5V" H 9050 4890 50  0000 C CNN
-F 2 "" H 9050 4750 50  0001 C CNN
-F 3 "" H 9050 4750 50  0001 C CNN
-	1    9050 4750
+P 9050 4800
+F 0 "#PWR013" H 9050 4650 50  0001 C CNN
+F 1 "+5V" H 9050 4940 50  0000 C CNN
+F 2 "" H 9050 4800 50  0001 C CNN
+F 3 "" H 9050 4800 50  0001 C CNN
+	1    9050 4800
 	0    1    1    0
 $EndComp
 $Comp
-L Conn_01x02 J1
+L CONN_01X02 J1
 U 1 1 5B353D06
 P 8850 4850

Commit message: Playing with via values to get advanced circuits to take it
Parts:
- J1: symbol CONN_01X02 -> Conn_01x02
- Q1: footprint TO_SOT_Packages_THT:TO-220_Vertical -> TO_SOT_Packages_SMD:SOT-666
Connections:
- wire segments 46 -> 50
- no-connect marks 88 -> 86
Changed lines of the file:
@@
 EESchema Schematic File Version 2
-LIBS:PowerBoard-rescue
 LIBS:power
 LIBS:device
@@
 F 0 "Q1" H 9300 5675 50  0000 L CNN
 F 1 "IRLB8721PBF" H 9300 5600 50  0000 L CNN
-F 2 "TO_SOT_Packages_THT:TO-220_Vertical" H 9300 5525 50  0001 L CIN
+F 2 "TO_SOT_Packages_SMD:SOT-666" H 9300 5525 50  0001 L CIN
 F 3 "" H 9050 5600 50  0001 L CNN
 	1    9050 5600
@@
 Wire Wire Line
 	9150 5400 9500 5400
-Text GLabel 9050 4900 2    60   Input ~ 0
+Text GLabel 9050 4850 2    60   Input ~ 0
 LineDeploymentDevice
 $Comp
 L +5V #PWR013
 U 1 1 5B353A83
-P 9050 4800
-F 0 "#PWR013" H 9050 4650 50  0001 C CNN
-F 1 "+5V" H 9050 4940 50  0000 C CNN
-F 2 "" H 9050 4800 50  0001 C CNN
-F 3 "" H 9050 4800 50  0001 C CNN
-	1    9050 4800
+P 9050 4750
+F 0 "#PWR013" H 9050 4600 50  0001 C CNN
+F 1 "+5V" H 9050 4890 50  0000 C CNN
+F 2 "" H 9050 4750 50  0001 C CNN
+F 3 "" H 9050 4750 50  0001 C CNN
+	1    9050 4750
 	0    1    1    0
 $EndComp
 $Comp
-L CONN_01X02 J1
+L Conn_01x02 J1
 U 1 1 5B353D06
 P 8850 4850
@@
 NoConn ~ 10500 8950
 NoConn ~ 10500 9050
-NoConn ~ 10500 9250
 NoConn ~ 10500 9850
 NoConn ~ 10500 9950
@@
 NoConn ~ 11000 9050
 NoConn ~ 11000 9150
-NoConn ~ 11000 9250
 NoConn ~ 11000 9950
 NoConn ~ 11000 10050
@@
 Connection ~ 8900 5650
 Connection ~ 8800 5850
+Wire Wire Line
+	10500 9250 10100 9250
+Wire Wire Line
+	10100 9250 10100 9150
+$Comp
+L +8V #PWR028
+U 1 1 5B3A7A86
+P 10100 9150
+F 0 "#PWR028" H 10100 9000 50  0001 C CNN
+F 1 "+8V" H 10100 9290 50  0000 C CNN
+F 2 "" H 10100 9150 50  0001 C CNN
+F 3 "" H 10100 9150 50  0001 C CNN
+	1    10100 9150
+	1    0    0    -1
+$EndComp
+Wire Wire Line
+	11000 9250 11400 9250
+Wire Wire Line
+	11400 9250 11400 9150
+$Comp
+L +8V #PWR029
+U 1 1 5B3A7C89
+P 11400 9150
+F 0 "#PWR029" H 11400 9000 50  0001 C CNN
+F 1 "+8V" H 11400 9290 50  0000 C CNN
+F 2 "" H 11400 9150 50  0001 C CNN
+F 3 "" H 11400 9150 50  0001 C CNN
+	1    11400 9150
+	1    0    0    -1
+$EndComp
 $EndSCHEMATC

Commit message: Update check
Parts:
- added D3: LED, LEDs:LED_0805, symbol LED
- added J2: ToResistor, Pin_Headers:Pin_Header_Straight_1x02_Pitch2.54mm, symbol Conn_01x02
- added Q2: IRLB8721PBF, TO_SOT_Packages_SMD:SOT-666, symbol IRLB8721PBF
- added R5: 51, Resistors_SMD:R_0805, symbol R
Connections:
- net labels added: SecondaryLineDeploymentDevice
- wire segments 50 -> 52
Other:
- moved on the sheet: D2, Q1, R4
Changed lines of the file:
@@
 LIBS:contrib
 LIBS:valves
-LIBS:pam
 LIBS:PowerBoard-cache
 EELAYER 25 0
@@
 L IRLB8721PBF Q1
 U 1 1 5B33FF0C
-P 9050 5600
-F 0 "Q1" H 9300 5675 50  0000 L CNN
-F 1 "IRLB8721PBF" H 9300 5600 50  0000 L CNN
-F 2 "TO_SOT_Packages_SMD:SOT-666" H 9300 5525 50  0001 L CIN
-F 3 "" H 9050 5600 50  0001 L CNN
-	1    9050 5600
+P 12250 5650
+F 0 "Q1" H 12500 5725 50  0000 L CNN
+F 1 "IRLB8721PBF" H 12500 5650 50  0000 L CNN
+F 2 "TO_SOT_Packages_SMD:SOT-666" H 12500 5575 50  0001 L CIN
+F 3 "" H 12250 5650 50  0001 L CNN
+	1    12250 5650
 	1    0    0    -1
 $EndComp
@@
 L GND #PWR012
 U 1 1 5B3400DC
-P 9150 5800
-F 0 "#PWR012" H 9150 5550 50  0001 C CNN
-F 1 "GND" H 9150 5650 50  0000 C CNN
-F 2 "" H 9150 5800 50  0001 C CNN
-F 3 "" H 9150 5800 50  0001 C CNN
-	1    9150 5800
-	1    0    0    -1
-$EndComp
-Wire Wire Line
-	9150 5400 9500 5400
-Text GLabel 9050 4850 2    60   Input ~ 0
-LineDeploymentDevice
+P 12350 5850
+F 0 "#PWR012" H 12350 5600 50  0001 C CNN
+F 1 "GND" H 12350 5700 50  0000 C CNN
+F 2 "" H 12350 5850 50  0001 C CNN
+F 3 "" H 12350 5850 50  0001 C CNN
+	1    12350 5850
+	1    0    0    -1
+$EndComp
+Wire Wire Line
+	12350 5450 12700 5450
+Text GLabel 12250 4900 2    60   Input ~ 0
+SecondaryLineDeploymentDevice
 $Comp
 L +5V #PWR013
 U 1 1 5B353A83
-P 9050 4750
-F 0 "#PWR013" H 9050 4600 50  0001 C CNN
-F 1 "+5V" H 9050 4890 50  0000 C CNN
-F 2 "" H 9050 4750 50  0001 C CNN
-F 3 "" H 9050 4750 50  0001 C CNN
-	1    9050 4750
+P 12250 4800
+F 0 "#PWR013" H 12250 4650 50  0001 C CNN
+F 1 "+5V" H 12250 4940 50  0000 C CNN
+F 2 "" H 12250 4800 50  0001 C CNN
+F 3 "" H 12250 4800 50  0001 C CNN
+	1    12250 4800
 	0    1    1    0
 $EndComp
@@
 L Conn_01x02 J1
 U 1 1 5B353D06
-P 8850 4850
-F 0 "J1" H 8850 4950 50  0000 C CNN
-F 1 "ToResistor" H 8850 4650 50  0000 C CNN
-F 2 "Pin_Headers:Pin_Header_Straight_1x02_Pitch2.54mm" H 8850 4850 50  0001 C CNN
-F 3 "" H 8850 4850 50  0001 C CNN
-	1    8850 4850
+P 12050 4900
+F 0 "J1" H 12050 5000 50  0000 C CNN
+F 1 "ToResistor" H 12050 4700 50  0000 C CNN
+F 2 "Pin_Headers:Pin_Header_Straight_1x02_Pitch2.54mm" H 12050 4900 50  0001 C CNN
+F 3 "" H 12050 4900 50  0001 C CNN
+	1    12050 4900
 	-1   0    0    1
 $EndComp
@@
 	1    0    0    -1
 $EndComp
-Text GLabel 9500 5400 2    60   Input ~ 0
-LineDeploymentDevice
+Text GLabel 12700 5450 2    60   Input ~ 0
+SecondaryLineDeploymentDevice
 $Comp
 L PAM2423A U1
@@
 NoConn ~ 9400 10650
 NoConn ~ 9400 9950
-Wire Wire Line
-	8900 5650 8900 5850
-Wire Wire Line
-	8900 5850 8800 5850
 $Comp
 L R R4
 U 1 1 5B36576A
-P 8650 5850
-F 0 "R4" V 8730 5850 50  0000 C CNN
-F 1 "51" V 8650 5850 50  0000 C CNN
-F 2 "Resistors_SMD:R_0805" V 8580 5850 50  0001 C CNN
-F 3 "" H 8650 5850 50  0001 C CNN
-	1    8650 5850
+P 11850 5900
+F 0 "R4" V 11930 5900 50  0000 C CNN
+F 1 "51" V 11850 5900 50  0000 C CNN
+F 2 "Resistors_SMD:R_0805" V 11780 5900 50  0001 C CNN
+F 3 "" H 11850 5900 50  0001 C CNN
+	1    11850 5900
 	0    1    1    0
 $EndComp
@@
 L LED D2
 U 1 1 5B3657B9
-P 8350 5850
-F 0 "D2" H 8350 5950 50  0000 C CNN
-F 1 "LED" H 8350 5750 50  0000 C CNN
-F 2 "LEDs:LED_0805" H 8350 5850 50  0001 C CNN
-F 3 "" H 8350 5850 50  0001 C CNN
-	1    8350 5850
+P 11550 5900
+F 0 "D2" H 11550 6000 50  0000 C CNN
+F 1 "LED" H 11550 5800 50  0000 C CNN
+F 2 "LEDs:LED_0805" H 11550 5900 50  0001 C CNN
+F 3 "" H 11550 5900 50  0001 C CNN
+	1    11550 5900
 	1    0    0    -1
 $EndComp
@@
 L GND #PWR027
 U 1 1 5B365800
-P 8200 5850
-F 0 "#PWR027" H 8200 5600 50  0001 C CNN
-F 1 "GND" H 8200 5700 50  0000 C CNN
-F 2 "" H 8200 5850 50  0001 C CNN
-F 3 "" H 8200 5850 50  0001 C CNN
-	1    8200 5850
+P 11400 5900
+F 0 "#PWR027" H 11400 5650 50  0001 C CNN
+F 1 "GND" H 11400 5750 50  0000 C CNN
+F 2 "" H 11400 5900 50  0001 C CNN
+F 3 "" H 11400 5900 50  0001 C CNN
+	1    11400 5900
 	0    1    1    0
 $EndComp
@@
 Sec_Deploy
 Wire Wire Line
-	8450 5650 8850 5650
-Text GLabel 8450 5650 0    60   Input ~ 0
+	11650 5700 12050 5700
+Text GLabel 11650 5700 0    60   Input ~ 0
 Pri_Deploy
-Text GLabel 8600 5650 1    60   Input ~ 0
+Text GLabel 11800 5700 1    60   Input ~ 0
 Sec_Deploy
-Connection ~ 8900 5650
-Connection ~ 8800 5850
+Connection ~ 12000 5900
 Wire Wire Line
 	10500 9250 10100 9250
@@
 	1    0    0    -1
 $EndComp
+$Comp
+L IRLB8721PBF Q2
+U 1 1 5B3BF4A7
+P 9150 5650
+F 0 "Q2" H 9400 5725 50  0000 L CNN
+F 1 "IRLB8721PBF" H 9400 5650 50  0000 L CNN
+F 2 "TO_SOT_Packages_SMD:SOT-666" H 9400 5575 50  0001 L CIN
+F 3 "" H 9150 5650 50  0001 L CNN
+	1    9150 5650
+	1    0    0    -1
+$EndComp
+$Comp
+L GND #PWR030
+U 1 1 5B3BF4AD
+P 9250 5850
+F 0 "#PWR030" H 9250 5600 50  0001 C CNN
+F 1 "GND" H 9250 5700 50  0000 C CNN
+F 2 "" H 9250 5850 50  0001 C CNN
+F 3 "" H 9250 5850 50  0001 C CNN
+	1    9250 5850
+	1    0    0    -1
+$EndComp
+Wire Wire Line
+	9250 5450 9600 5450
+Text GLabel 9150 4900 2    60   Input ~ 0
+LineDeploymentDevice
+$Comp
+L +5V #PWR031
+U 1 1 5B3BF4B5
+P 9150 4800
+F 0 "#PWR031" H 9150 4650 50  0001 C CNN
+F 1 "+5V" H 9150 4940 50  0000 C CNN
+F 2 "" H 9150 4800 50  0001 C CNN
+F 3 "" H 9150 4800 50  0001 C CNN
+	1    9150 4800
+	0    1    1    0
+$EndComp
+$Comp
+L Conn_01x02 J2
+U 1 1 5B3BF4BB
+P 8950 4900
+F 0 "J2" H 8950 5000 50  0000 C CNN
+F 1 "ToResistor" H 8950 4700 50  0000 C CNN
+F 2 "Pin_Headers:Pin_Header_Straight_1x02_Pitch2.54mm" H 8950 4900 50  0001 C CNN
+F 3 "" H 8950 4900 50  0001 C CNN
+	1    8950 4900
+	-1   0    0    1
+$EndComp
+Text GLabel 9600 5450 2    60   Input ~ 0
+LineDeploymentDevice
+$Comp
+L R R5
+U 1 1 5B3BF4C4
+P 8750 5900
+F 0 "R5" V 8830 5900 50  0000 C CNN
+F 1 "51" V 8750 5900 50  0000 C CNN
+F 2 "Resistors_SMD:R_0805" V 8680 5900 50  0001 C CNN
+F 3 "" H 8750 5900 50  0001 C CNN
+	1    8750 5900
+	0    1    1    0
+$EndComp
+$Comp
+L LED D3
+U 1 1 5B3BF4CA
+P 8450 5900
+F 0 "D3" H 8450 6000 50  0000 C CNN
+F 1 "LED" H 8450 5800 50  0000 C CNN
+F 2 "LEDs:LED_0805" H 8450 5900 50  0001 C CNN
+F 3 "" H 8450 5900 50  0001 C CNN
+	1    8450 5900
+	1    0    0    -1
+$EndComp
+$Comp
+L GND #PWR032
+U 1 1 5B3BF4D0
+P 8300 5900
+F 0 "#PWR032" H 8300 5650 50  0001 C CNN
+F 1 "GND" H 8300 5750 50  0000 C CNN
+F 2 "" H 8300 5900 50  0001 C CNN
+F 3 "" H 8300 5900 50  0001 C CNN
+	1    8300 5900
+	0    1    1    0
+$EndComp
+Wire Wire Line
+	8550 5700 8950 5700
+Text GLabel 8550 5700 0    60   Input ~ 0
+Pri_Deploy
+Text GLabel 8700 5700 1    60   Input ~ 0
+Sec_Deploy
+Connection ~ 8900 5900
+Wire Wire Line
+	12000 5900 12000 5700
+Connection ~ 12000 5700
+Wire Wire Line
+	8900 5900 8900 5700
+Connection ~ 8900 5700
 $EndSCHEMATC

Commit message: Fixed PC104 conflicts and added i2c debug
Parts:
- added J3: I2C_Debug, Socket_Strips:Socket_Strip_Angled_1x02_Pitch2.54mm, symbol conn:Conn_01x02
- C1, C8: symbol CP1 -> device:CP1
- C2, C3, C4, C5, C6, C7: symbol C -> device:C
- D1: symbol D_Zener -> device:D_Zener
- D2, D3: symbol LED -> device:LED
- H1, H2: symbol CONN_02X26 -> PowerBoard-rescue:CONN_02X26
- J1, J2: symbol Conn_01x02 -> conn:Conn_01x02
- L1: symbol L -> device:L
- Q1, Q2: symbol IRLB8721PBF -> transistors:IRLB8721PBF
- R1, R2, R3, R4, R5: symbol R -> device:R
Connections:
- net labels added: I2C_SCL, I2C_SDA
- wire segments 52 -> 74
- no-connect marks 86 -> 82
